Commit message: Sim it works!

File: description/urdf/lidar_sick_lms_291.urdf.xacro (robot description, xacro)
@@ -11,5 +11,5 @@
       <visual>
         <geometry>
-          <mesh filename="$(find caddy_ai2_ros2_control_sensors_lidar_sick_lms_291)/meshes/dae/SICK_LMS291-S05.dae" scale="1 1 1"/>
+          <mesh filename="file://$(find caddy_ai2_ros2_control_sensors_lidar_sick_lms_291)/meshes/dae/SICK_LMS291-S05.dae" scale="1 1 1"/>
         </geometry>
       </visual>
